File: Electronics documents/Spinning_display_KiCad/Spinning_display.kicad_sch (KiCad schematic)
At the start: 52 parts

Commit message: Documentation update
Other:
- company: (none) -> UVic-UCC
- title: (none) -> Spinning LED Display
Changed lines of the file:
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@@
 (kicad_sch (version 20211123) (generator eeschema)
   (paper "A4")
+  (title_block
+    (title "Spinning LED Display")
+    (company "UVic-UCC")
+  )
   (junction (at 74.93 129.54) (diameter 0) (color 0 0 0 0)
   )
